Commit message: Modifications to switch from ROS Fuerte to ROS Noetic

File: youbot_ws/src/ros_stacks/youbot-ros-pkg/youbot_common/youbot_description/robots/youbot-sensors.urdf.xacro (robot description, xacro)
@@ -7,17 +7,17 @@
   <!-- The following included files set up definitions of parts of the robot body -->
   <!-- misc common stuff? -->
-  <include filename="$(find youbot_description)/urdf/common.xacro" />
+  <xacro:include filename="$(find youbot_description)/urdf/common.xacro" />
   <!-- youbot base -->
-  <include filename="$(find youbot_description)/urdf/youbot_base/base.urdf.xacro" />
+  <xacro:include filename="$(find youbot_description)/urdf/youbot_base/base.urdf.xacro" />
   <!-- youbot plate -->
-  <include filename="$(find youbot_description)/urdf/youbot_plate/plate.urdf.xacro" />
+  <xacro:include filename="$(find youbot_description)/urdf/youbot_plate/plate.urdf.xacro" />
   <!-- youbot arm -->
-  <include filename="$(find youbot_description)/urdf/youbot_arm/arm.urdf.xacro"/>
+  <xacro:include filename="$(find youbot_description)/urdf/youbot_arm/arm.urdf.xacro"/>
   <!-- youbot gripper -->
-  <include filename="$(find youbot_description)/urdf/youbot_gripper/gripper.urdf.xacro" />
+  <xacro:include filename="$(find youbot_description)/urdf/youbot_gripper/gripper.urdf.xacro" />
   <!-- generic simulator_gazebo plugins for starting mechanism control, ros time, ros battery -->
-  <include filename="$(find youbot_description)/gazebo/gazebo.urdf.xacro" />
+  <xacro:include filename="$(find youbot_description)/gazebo/gazebo.urdf.xacro" />
   <!-- materials for visualization -->
-  <include filename="$(find youbot_description)/urdf/materials.urdf.xacro" />
+  <xacro:include filename="$(find youbot_description)/urdf/materials.urdf.xacro" />
   <!-- Now we can start using the macros included above to define the actual youbot -->
   <!-- The first use of a macro.  This one was defined in base.urdf.xacro above.
@@ -40,10 +40,10 @@
   </xacro:youbot_gripper>
   <!-- BRSU SPECIFIC STUFF -->
-  <include filename="$(find youbot_description)/urdf/updated_materials.urdf.xacro" />
-  <include filename="$(find youbot_description)/urdf/misc/sensor_angle.urdf.xacro" />
-  <include filename="$(find youbot_description)/urdf/misc/cam3d_tower.urdf.xacro" />
-  <include filename="$(find youbot_description)/urdf/sensors/kinect_camera.urdf.xacro" />
-  <include filename="$(find youbot_description)/urdf/sensors/microsoft_lifecam.urdf.xacro" />
-  <include filename="$(find youbot_description)/urdf/sensors/asus_xtion_camera.urdf.xacro" />
+  <xacro:include filename="$(find youbot_description)/urdf/updated_materials.urdf.xacro" />
+  <xacro:include filename="$(find youbot_description)/urdf/misc/sensor_angle.urdf.xacro" />
+  <xacro:include filename="$(find youbot_description)/urdf/misc/cam3d_tower.urdf.xacro" />
+  <xacro:include filename="$(find youbot_description)/urdf/sensors/kinect_camera.urdf.xacro" />
+  <xacro:include filename="$(find youbot_description)/urdf/sensors/microsoft_lifecam.urdf.xacro" />
+  <xacro:include filename="$(find youbot_description)/urdf/sensors/asus_xtion_camera.urdf.xacro" />
   <!-- base laser rear -->
   <xacro:hokuyo_urg04_laser name="base_laser_rear" parent="base" ros_topic="scan_rear" update_rate="10" min_angle="-1.57" max_angle="1.57">

File: youbot_ws/src/ros_stacks/youbot-ros-pkg/youbot_common/youbot_description/robots/youbot.urdf.xacro (robot description, xacro)
@@ -7,17 +7,17 @@
   <!-- The following included files set up definitions of parts of the robot body -->
   <!-- misc common stuff? -->
-  <include filename="$(find youbot_description)/urdf/common.xacro" />
+  <xacro:include filename="$(find youbot_description)/urdf/common.xacro" />
   <!-- youbot base -->
-  <include filename="$(find youbot_description)/urdf/youbot_base/base.urdf.xacro" />
+  <xacro:include filename="$(find youbot_description)/urdf/youbot_base/base.urdf.xacro" />
   <!-- youbot plate -->
-  <include filename="$(find youbot_description)/urdf/youbot_plate/plate.urdf.xacro" />
+  <xacro:include filename="$(find youbot_description)/urdf/youbot_plate/plate.urdf.xacro" />
   <!-- youbot arm -->
-  <include filename="$(find youbot_description)/urdf/youbot_arm/arm.urdf.xacro"/>
+  <xacro:include filename="$(find youbot_description)/urdf/youbot_arm/arm.urdf.xacro"/>
   <!-- youbot gripper -->
-  <include filename="$(find youbot_description)/urdf/youbot_gripper/gripper.urdf.xacro" />
+  <xacro:include filename="$(find youbot_description)/urdf/youbot_gripper/gripper.urdf.xacro" />
   <!-- generic simulator_gazebo plugins for starting mechanism control, ros time, ros battery -->
-  <include filename="$(find youbot_description)/gazebo/gazebo.urdf.xacro" />
+  <xacro:include filename="$(find youbot_description)/gazebo/gazebo.urdf.xacro" />
   <!-- materials for visualization -->
-  <include filename="$(find youbot_description)/urdf/materials.urdf.xacro" />
+  <xacro:include filename="$(find youbot_description)/urdf/materials.urdf.xacro" />
   <!-- Now we can start using the macros included above to define the actual youbot -->
   <!-- The first use of a macro.  This one was defined in base.urdf.xacro above.

File: youbot_ws/src/ros_stacks/youbot-ros-pkg/youbot_common/youbot_description/robots/youbot_dual_arm.urdf.xacro (robot description, xacro)
@@ -7,17 +7,17 @@
   <!-- The following included files set up definitions of parts of the robot body -->
   <!-- misc common stuff? -->
-  <include filename="$(find youbot_description)/urdf/common.xacro" />
+  <xacro:include filename="$(find youbot_description)/urdf/common.xacro" />
   <!-- youbot base -->
-  <include filename="$(find youbot_description)/urdf/youbot_base/base.urdf.xacro" />
+  <xacro:include filename="$(find youbot_description)/urdf/youbot_base/base.urdf.xacro" />
   <!-- youbot plate -->
-  <include filename="$(find youbot_description)/urdf/youbot_plate/plate.urdf.xacro" />
+  <xacro:include filename="$(find youbot_description)/urdf/youbot_plate/plate.urdf.xacro" />
   <!-- youbot arm -->
-  <include filename="$(find youbot_description)/urdf/youbot_arm/arm.urdf.xacro"/>
+  <xacro:include filename="$(find youbot_description)/urdf/youbot_arm/arm.urdf.xacro"/>
   <!-- youbot gripper -->
-  <include filename="$(find youbot_description)/urdf/youbot_gripper/gripper.urdf.xacro" />
+  <xacro:include filename="$(find youbot_description)/urdf/youbot_gripper/gripper.urdf.xacro" />
   <!-- generic simulator_gazebo plugins for starting mechanism control, ros time, ros battery -->
-  <include filename="$(find youbot_description)/gazebo/gazebo.urdf.xacro" />
+  <xacro:include filename="$(find youbot_description)/gazebo/gazebo.urdf.xacro" />
   <!-- materials for visualization -->
-  <include filename="$(find youbot_description)/urdf/materials.urdf.xacro" />
+  <xacro:include filename="$(find youbot_description)/urdf/materials.urdf.xacro" />
   <!-- Now we can start using the macros included above to define the actual youbot -->
   <!-- The first use of a macro.  This one was defined in base.urdf.xacro above.

File: youbot_ws/src/ros_stacks/youbot-ros-pkg/youbot_common/youbot_description/urdf/common.xacro (robot description, xacro)
@@ -1,9 +1,9 @@
 <?xml version="1.0"?>
-<robot>
-	<property name="M_PI" value="3.1415926535897931" />
+<robot xmlns:xacro="http://ros.org/wiki/xacro">
+	<xacro:property name="M_PI" value="3.1415926535897931" />
 	<!-- Casters -->
-	<property name="cal_caster_fl" value="0.0" />
-	<property name="cal_caster_fr" value="0.0" />
-	<property name="cal_caster_bl" value="0.0" />
-	<property name="cal_caster_br" value="0.0" />
+	<xacro:property name="cal_caster_fl" value="0.0" />
+	<xacro:property name="cal_caster_fr" value="0.0" />
+	<xacro:property name="cal_caster_bl" value="0.0" />
+	<xacro:property name="cal_caster_br" value="0.0" />
 </robot>

File: youbot_ws/src/ros_stacks/youbot-ros-pkg/youbot_common/youbot_description/urdf/misc/cam3d_tower.urdf.xacro (robot description, xacro)
@@ -4,7 +4,7 @@
        xmlns:interface="http://playerstage.sourceforge.net/gazebo/xmlschema/#interface"
        xmlns:xacro="http://ros.org/wiki/xacro">
-  <property name="cam3d_tower_height" value="0.49" />
-  <property name="cam3d_tower_width" value="0.03" />
-  <property name="cam3d_tower_depth" value="0.03" />
+  <xacro:property name="cam3d_tower_height" value="0.49" />
+  <xacro:property name="cam3d_tower_width" value="0.03" />
+  <xacro:property name="cam3d_tower_depth" value="0.03" />
   <xacro:macro name="cam3d_tower" params="name parent *origin">
   	<link name="${name}_link">

File: youbot_ws/src/ros_stacks/youbot-ros-pkg/youbot_common/youbot_description/urdf/misc/sensor_angle.urdf.xacro (robot description, xacro)
@@ -4,7 +4,7 @@
        xmlns:interface="http://playerstage.sourceforge.net/gazebo/xmlschema/#interface"
        xmlns:xacro="http://ros.org/wiki/xacro">
-	<property name="sensor_angle_width"  value="0.097" />
-	<property name="sensor_angle_height" value="0.0015" />
-	<property name="sensor_angle_depth"  value="0.0625" />
+	<xacro:property name="sensor_angle_width"  value="0.097" />
+	<xacro:property name="sensor_angle_height" value="0.0015" />
+	<xacro:property name="sensor_angle_depth"  value="0.0625" />
 	<xacro:macro name="sensor_angle" params="name parent *origin">
 		<link name="${name}_part1_link">

File: youbot_ws/src/ros_stacks/youbot-ros-pkg/youbot_common/youbot_description/urdf/sensors/asus_xtion_camera.urdf.xacro (robot description, xacro)
@@ -2,6 +2,6 @@
 <root xmlns:xacro="http://playerstage.sourceforge.net/gazebo/xmlschema/#interface">
   <include filename="$(find youbot_description)/urdf/sensors/asus_xtion_camera.gazebo.xacro" />
-  <property name="eye_x_offset" value="0.03" />
-  <property name="eye_y_offset" value="0.035" />
+  <xacro:property name="eye_x_offset" value="0.03" />
+  <xacro:property name="eye_y_offset" value="0.035" />
   <xacro:macro name="asus_xtion_eye" params="suffix parent *origin">
 	<link name="${parent}_${suffix}_frame">

File: youbot_ws/src/ros_stacks/youbot-ros-pkg/youbot_common/youbot_description/urdf/youbot_arm/arm.urdf.xacro (robot description, xacro)
@@ -4,7 +4,7 @@
         xmlns:interface="http://playerstage.sourceforge.net/gazebo/xmlschema/#interface"
         xmlns:xacro="http://ros.org/wiki/xacro">
-	<include filename="$(find youbot_description)/urdf/youbot_arm/arm.gazebo.xacro" />
-	<include filename="$(find youbot_description)/urdf/youbot_arm/arm.transmission.xacro" />
-        <include filename="$(find youbot_description)/urdf/youbot_arm/limits.urdf.xacro" />
+	<xacro:include filename="$(find youbot_description)/urdf/youbot_arm/arm.gazebo.xacro" />
+	<xacro:include filename="$(find youbot_description)/urdf/youbot_arm/arm.transmission.xacro" />
+    <xacro:include filename="$(find youbot_description)/urdf/youbot_arm/limits.urdf.xacro" />
 	<xacro:macro name="youbot_arm" params="parent name *origin">
 		<!-- joint between base_link and arm_0_link -->

File: youbot_ws/src/ros_stacks/youbot-ros-pkg/youbot_common/youbot_description/urdf/youbot_arm/limits.urdf.xacro (robot description, xacro)
@@ -1,25 +1,25 @@
 <?xml version="1.0"?>
-<robot xmlns:xacro="http://ros.org/wiki/xacro">>
+<robot xmlns:xacro="http://ros.org/wiki/xacro">
 	<!-- common properties -->
-	<property name="M_PI" value="3.1415926535897931" />
-        <property name="threshold" value="0.01" />
+	<xacro:property name="M_PI" value="3.1415926535897931" />
+    <xacro:property name="threshold" value="0.01" />
 	<!-- arm limits positions (deg) -->
-	<property name="joint_1_limit" value="${M_PI * (169 + 169) / 180}" />
-	<property name="joint_2_limit" value="${M_PI * (90 + 65) / 180}" />
-	<property name="joint_3_limit" value="${M_PI * (146 + 151) / 180}" />
-	<property name="joint_4_limit" value="${M_PI * (102.5 + 102.5) / 180}" />
-	<property name="joint_5_limit" value="${M_PI * (167.5 + 167.5) / 180}" />
-        <property name="joint_1_limit_soft" value="${M_PI * (169 + 169) / 180 - threshold}" />
-	<property name="joint_2_limit_soft" value="${M_PI * (90 + 65) / 180 - threshold}" />
-	<property name="joint_3_limit_soft" value="${M_PI * (146 + 151) / 180 - threshold}" />
-	<property name="joint_4_limit_soft" value="${M_PI * (102.5 + 102.5) / 180 - threshold}" />
-	<property name="joint_5_limit_soft" value="${M_PI * (167.5 + 167.5) / 180 - threshold}" />
+	<xacro:property name="joint_1_limit" value="${M_PI * (169 + 169) / 180}" />
+	<xacro:property name="joint_2_limit" value="${M_PI * (90 + 65) / 180}" />
+	<xacro:property name="joint_3_limit" value="${M_PI * (146 + 151) / 180}" />
+	<xacro:property name="joint_4_limit" value="${M_PI * (102.5 + 102.5) / 180}" />
+	<xacro:property name="joint_5_limit" value="${M_PI * (167.5 + 167.5) / 180}" />
+    <xacro:property name="joint_1_limit_soft" value="${M_PI * (169 + 169) / 180 - threshold}" />
+	<xacro:property name="joint_2_limit_soft" value="${M_PI * (90 + 65) / 180 - threshold}" />
+	<xacro:property name="joint_3_limit_soft" value="${M_PI * (146 + 151) / 180 - threshold}" />
+	<xacro:property name="joint_4_limit_soft" value="${M_PI * (102.5 + 102.5) / 180 - threshold}" />
+	<xacro:property name="joint_5_limit_soft" value="${M_PI * (167.5 + 167.5) / 180 - threshold}" />
 	<!-- dynamic properties : mass (kg) Alu data sheet -->
-	<property name="link_0_mass" value="0.845" />
-	<property name="link_1_mass" value="2.412" />
-	<property name="link_2_mass" value="1.155" />
-	<property name="link_3_mass" value="0.934" />
-	<property name="link_4_mass" value="0.877" />
-	<property name="link_5_mass" value="0.251" />
+	<xacro:property name="link_0_mass" value="0.845" />
+	<xacro:property name="link_1_mass" value="2.412" />
+	<xacro:property name="link_2_mass" value="1.155" />
+	<xacro:property name="link_3_mass" value="0.934" />
+	<xacro:property name="link_4_mass" value="0.877" />
+	<xacro:property name="link_5_mass" value="0.251" />
 	<!--<property name="link_0_mass" value="0.845" />
 	<property name="link_1_mass" value="0.1" />

File: youbot_ws/src/ros_stacks/youbot-ros-pkg/youbot_common/youbot_description/urdf/youbot_base/base.transmission.xacro (robot description, xacro)
@@ -4,7 +4,6 @@
        xmlns:interface="http://playerstage.sourceforge.net/gazebo/xmlschema/#interface"
        xmlns:xacro="http://ros.org/wiki/xacro">
-	<property name="wheel_mechanical_reduction" value="${624/35 * 80/18}" />
-	<property name="caster_mechanical_reduction" value="${624/35 * 80/18}" />
-  	<property name="" value="0.360" />
+	<xacro:property name="wheel_mechanical_reduction" value="${624/35 * 80/18}" />
+	<xacro:property name="caster_mechanical_reduction" value="${624/35 * 80/18}" />
 	<xacro:macro name="youbot_base_transmission">
 	<!-- front left wheel -->
