Commit message: Modifications to switch from ROS Fuerte to ROS Noetic

File: youbot_ws/src/ros_stacks/youbot-ros-pkg/youbot_common/youbot_description/urdf/youbot_base/base.urdf.xacro (robot description, xacro)
@@ -4,286 +4,286 @@
         xmlns:interface="http://playerstage.sourceforge.net/gazebo/xmlschema/#interface"
         xmlns:xacro="http://ros.org/wiki/xacro">
-	<!-- sensors -->
-	<include filename="$(find youbot_description)/urdf/sensors/hokuyo_urg04_laser.urdf.xacro"/>
-	<include filename="$(find youbot_description)/urdf/youbot_base/base.gazebo.xacro" />
-	<include filename="$(find youbot_description)/urdf/youbot_base/base.transmission.xacro" />
- 	<!-- simplified box collision geometry for base -->
-  	<property name="base_size_x" value="0.570" />
-  	<property name="base_size_y" value="0.360" />
-  	<property name="base_size_z" value="0.100" />
-	<property name="base_mass" value="22.0" />
-	<property name="caster_offset_x" value="0.228"  />
-  	<property name="caster_offset_y" value="0.158"  />
-  	<property name="caster_offset_z" value="-0.034" />
-	<property name="caster_mass" value="0.1" />
-	<property name="wheel_offset_x" value="0.0"  />
-  	<property name="wheel_offset_y" value="0.0"  />
-  	<property name="wheel_offset_z" value="0.0" />
-	<property name="wheel_mass" value="0.4" />
-	<property name="wheel_radius" value="0.05" />
-	<property name="wheel_length" value="0.005" />
-	<property name="caster_joint_damping" value="1.0" />
-	<property name="caster_joint_friction" value="1.0" />
-	<property name="caster_joint_effort" value="30" />
-	<property name="caster_joint_velocity" value="10" />
-	<property name="caster_joint_safety_k_velocity" value="10.0" />
-	<property name="wheel_joint_damping" value="1.0" />
-	<property name="wheel_joint_friction" value="1.0" />
-	<property name="wheel_joint_effort" value="30" />
-	<property name="wheel_joint_velocity" value="10" />
-	<property name="wheel_joint_safety_k_velocity" value="10.0" />
-	<xacro:macro name="youbot_base" params="name">
-		<link name="${name}_footprint">
-      			<inertial>
-        			<mass value="0.1" />
-        			<origin xyz="0 0 ${-base_size_z / 2.0}" rpy="0 0 0" />
-        			<inertia ixx="1.0" ixy="0.0" ixz="0.0"
-                 			iyy="1.0" iyz="0.0" izz="1.0" />
-      				</inertial>
-      			<visual>
-        			<origin xyz="0 0 0" rpy="0 0 0" />
-        			<geometry>
-          				<box size="0.001 0.001 0.001" />
-        			</geometry>
-               			<material name="Red" />
-      			</visual>
-      			<collision>
-        			<origin xyz="0 0 ${-base_size_z / 2.0}" rpy="0 0 0" />
-        			<geometry>
-          				<box size="0.001 0.001 0.001" />
-        			</geometry>
-      			</collision>
-    		</link>
-    		<joint name="${name}_footprint_joint" type="fixed">
-      			<origin xyz="0 0 0" rpy="0 0 0" />
-      			<child link="${name}_link" />
-      			<parent link="${name}_footprint"/>
-    		</joint>
-		<link name="${name}_link">
-      			<inertial>
-        			<mass value="${base_mass}" />
-        			<origin xyz="0 0 0" />
-        			<inertia ixx="5.652232699207" ixy="-0.009719934438" ixz="1.293988226423"
-                 			iyy="5.669473158652" iyz="-0.007379583694" izz="3.683196351726" />
-      				</inertial>
-      			<visual>
-        			<origin xyz="0 0 0" rpy="0 0 0" />
-        			<geometry>
-          				<mesh filename="package://youbot_description/meshes/youbot_base/base.dae"/>
-        			</geometry>
-        			<material name="DarkGrey"/>
-      			</visual>
-      			<collision>
-        			<origin xyz="0 0 0" rpy="0 0 0" />
-        			<geometry>
-          				<!--<box size="${base_size_x} ${base_size_y} ${base_size_z}" />-->
-					<mesh filename="package://youbot_description/meshes/youbot_base/base_convex.dae"/>
-	       			</geometry>
-      			</collision>
-    		</link>
-		<!-- base laser front -->
-    		<xacro:hokuyo_urg04_laser name="${name}_laser_front" parent="${name}" ros_topic="scan_front" update_rate="10" min_angle="-1.57" max_angle="1.57" >
-     			 <origin xyz="0.3 0 -0.03" rpy="0 0 0" />
-    		</xacro:hokuyo_urg04_laser>
-	<!-- front left wheel -->
-		<joint name="caster_joint_fl" type="continuous">
-			<origin xyz="${caster_offset_x} ${caster_offset_y} ${caster_offset_z}" rpy="0 0 0" />
-      			<axis xyz="0 0 1" />
-      			<limit effort="${caster_joint_effort}" velocity="${caster_joint_velocity}"/>
-      			<dynamics damping="${caster_joint_damping}" friction="${caster_joint_friction}" />
-			<safety_controller k_velocity="${caster_joint_safety_k_velocity}" />
-			<parent link="${name}_link"/>
-      			<child link="caster_link_fl" />
-    		</joint>
-		<link name="caster_link_fl">
-      			<inertial>
-        			<mass value="${caster_mass}" />
-        			<origin xyz="0 0 0" />
-        			<inertia  ixx="0.012411765597" ixy="-0.000711733678" ixz="0.00050272983"
-                  			iyy="0.015218160428" iyz="-0.000004273467" izz="0.011763977943" />
-      			</inertial>
-   		</link>
-		<joint name="wheel_joint_fl" type="continuous">
-      			<axis xyz="0 1 0" />
-      			<limit effort="${wheel_joint_effort}" velocity="${wheel_joint_velocity}"/>
-            		<origin xyz="${wheel_offset_x} ${wheel_offset_y} ${wheel_offset_z}" rpy="0 0 0" />
-      			<parent link="caster_link_fl"/>
-			<dynamics damping="${wheel_joint_damping}" friction="${wheel_joint_friction}" />
-			<safety_controller k_velocity="${wheel_joint_safety_k_velocity}" />
-      			<child link="wheel_link_fl"/>
-     		</joint>
-    		<link name="wheel_link_fl">
-      			<inertial>
-        		<mass value="${wheel_mass}" />
-        		<origin xyz="0 0 0" />
-       			<inertia  ixx="0.012411765597" ixy="-0.000711733678" ixz="0.00050272983"
-                  		iyy="0.015218160428" iyz="-0.000004273467" izz="0.011763977943" />
-      			</inertial>
-      			<visual>
-        			<origin xyz="0 0 0" rpy="0 0 0" />
-					<!--<mesh filename="package://youbot_description/meshes/youbot_base/youbot_wheel.stl" />-->
-				<geometry>
-					<sphere radius="${wheel_radius}"/>
-				</geometry>
-       				<material name="Orange" />
-      			</visual>
-      			<collision>
-        			<origin xyz="0 0 0" rpy="${M_PI/2} 0 0" />
-        			<geometry>
-        		       		<cylinder radius="${wheel_radius}" length="${wheel_radius}" />
-        	       		</geometry>
-      			</collision>
-    		</link>
-	<!-- front right wheel -->
-		<joint name="caster_joint_fr" type="continuous">
-			<origin xyz="${caster_offset_x} ${-caster_offset_y} ${caster_offset_z}" rpy="0 0 0" />
-      			<axis xyz="0 0 1" />
-      			<limit effort="${caster_joint_effort}" velocity="${caster_joint_velocity}"/>
-      			<dynamics damping="${caster_joint_damping}" friction="${caster_joint_friction}" />
-			<safety_controller k_velocity="${caster_joint_safety_k_velocity}" />
-			<parent link="${name}_link"/>
-      			<child link="caster_link_fr" />
-    		</joint>
-		<link name="caster_link_fr">
-      			<inertial>
-        			<mass value="${caster_mass}" />
-        			<origin xyz="0 0 0" />
-        			<inertia  ixx="0.012411765597" ixy="-0.000711733678" ixz="0.00050272983"
-                  			iyy="0.015218160428" iyz="-0.000004273467" izz="0.011763977943" />
-      				</inertial>
-   		</link>
-		<joint name="wheel_joint_fr" type="continuous">
-      			<axis xyz="0 1 0" />
-      			<limit effort="${wheel_joint_effort}" velocity="${wheel_joint_velocity}"/>
-            		<dynamics damping="${wheel_joint_damping}" friction="${wheel_joint_friction}" />
-			<safety_controller k_velocity="${wheel_joint_safety_k_velocity}" />
-      			<origin xyz="${wheel_offset_x} ${wheel_offset_y} ${wheel_offset_z}" rpy="0 0 0" />
-      			<parent link="caster_link_fr"/>
-      			<child link="wheel_link_fr"/>
-     		</joint>
-    		<link name="wheel_link_fr">
-      			<inertial>
-        		<mass value="${wheel_mass}" />
-        		<origin xyz="0 0 0" />
-       			<inertia  ixx="0.012411765597" ixy="-0.000711733678" ixz="0.00050272983"
-                  		iyy="0.015218160428" iyz="-0.000004273467" izz="0.011763977943" />
-      			</inertial>
-      			<visual>
-        			<origin xyz="0 0 0" rpy="0 0 0" />
-				<geometry>
-          				<!--<mesh filename="package://youbot_description/meshes/youbot_base/youbot_wheel.stl" />-->
-					<sphere radius="${wheel_radius}"/>
-        			</geometry>
-       				<material name="Orange" />
-      			</visual>
-      			<collision>
-        			<origin xyz="0 0 0" rpy="${M_PI/2} 0 0" />
-        			<geometry>
-        		       		<cylinder radius="${wheel_radius}" length="${wheel_radius}" />
-        	       		</geometry>
-      			</collision>
-    		</link>
-	<!-- back left wheel -->
-		<joint name="caster_joint_bl" type="continuous">
-			<origin xyz="${-caster_offset_x} ${caster_offset_y} ${caster_offset_z}" rpy="0 0 0" />
-      			<axis xyz="0 0 1" />
-      			<limit effort="${caster_joint_effort}" velocity="${caster_joint_velocity}"/>
-      			<dynamics damping="${caster_joint_damping}" friction="${caster_joint_friction}" />
-			<safety_controller k_velocity="${caster_joint_safety_k_velocity}" />
-			<parent link="${name}_link"/>
-      			<child link="caster_link_bl" />
-    		</joint>
-		<link name="caster_link_bl">
-      			<inertial>
-        			<mass value="${caster_mass}" />
-        			<origin xyz="0 0 0" />
-        			<inertia  ixx="0.012411765597" ixy="-0.000711733678" ixz="0.00050272983"
-                  			iyy="0.015218160428" iyz="-0.000004273467" izz="0.011763977943" />
-      				</inertial>
-   		</link>
-		<joint name="wheel_joint_bl" type="continuous">
-      			<axis xyz="0 1 0" />
-      			<limit effort="10" velocity="10"/>
-			<limit effort="${wheel_joint_effort}" velocity="${wheel_joint_velocity}"/>
-			<dynamics damping="${wheel_joint_damping}" friction="${wheel_joint_friction}" />
-			<safety_controller k_velocity="${wheel_joint_safety_k_velocity}" />
-      			<origin xyz="${wheel_offset_x} ${wheel_offset_y} ${wheel_offset_z}" rpy="0 0 0" />
-      			<parent link="caster_link_bl"/>
-      			<child link="wheel_link_bl"/>
-     		</joint>
-    		<link name="wheel_link_bl">
-      			<inertial>
-        		<mass value="${wheel_mass}" />
-        		<origin xyz="0 0 0" />
-       			<inertia  ixx="0.012411765597" ixy="-0.000711733678" ixz="0.00050272983"
-                  		iyy="0.015218160428" iyz="-0.000004273467" izz="0.011763977943" />
-      			</inertial>
-      			<visual>
-        			<origin xyz="0 0 0" rpy="0 0 0" />
-				<geometry>
-          				<!--<mesh filename="package://youbot_description/meshes/youbot_base/youbot_wheel.stl" />-->
-					<sphere radius="${wheel_radius}"/>
-        			</geometry>
-       				<material name="Orange" />
-      			</visual>
-      			<collision>
-        			<origin xyz="0 0 0" rpy="${M_PI/2} 0 0" />
-        			<geometry>
-        		       		<cylinder radius="${wheel_radius}" length="${wheel_radius}" />
-        	       		</geometry>
-      			</collision>
-    		</link>
-	<!-- back right wheel -->
-		<joint name="caster_joint_br" type="continuous">
-			<origin xyz="${-caster_offset_x} ${-caster_offset_y} ${caster_offset_z}" rpy="0 0 0" />
-      			<axis xyz="0 0 1" />
-      			<limit effort="${caster_joint_effort}" velocity="${caster_joint_velocity}"/>
-      			<dynamics damping="${caster_joint_damping}" friction="${caster_joint_friction}" />
-			<safety_controller k_velocity="${caster_joint_safety_k_velocity}" />
-			<parent link="${name}_link"/>
-      			<child link="caster_link_br" />
-    		</joint>
-		<link name="caster_link_br">
-      			<inertial>
-        			<mass value="${caster_mass}" />
-        			<origin xyz="0 0 0" />
-        			<inertia  ixx="0.012411765597" ixy="-0.000711733678" ixz="0.00050272983"
-                  			iyy="0.015218160428" iyz="-0.000004273467" izz="0.011763977943" />
-      				</inertial>
-   		</link>
-		<joint name="wheel_joint_br" type="continuous">
-      			<axis xyz="0 1 0" />
-      			<limit effort="${wheel_joint_effort}" velocity="${wheel_joint_velocity}"/>
-            		<dynamics damping="${wheel_joint_damping}" friction="${wheel_joint_friction}" />
-			<safety_controller k_velocity="${wheel_joint_safety_k_velocity}" />
-      			<origin xyz="${wheel_offset_x} ${wheel_offset_y} ${wheel_offset_z}" rpy="0 0 0" />
-      			<parent link="caster_link_br"/>
-      			<child link="wheel_link_br"/>
-     		</joint>
-    		<link name="wheel_link_br">
-      			<inertial>
-        		<mass value="${wheel_mass}" />
-        		<origin xyz="0 0 0" />
-       			<inertia  ixx="0.012411765597" ixy="-0.000711733678" ixz="0.00050272983"
-                  		iyy="0.015218160428" iyz="-0.000004273467" izz="0.011763977943" />
-      			</inertial>
-      			<visual>
-        			<origin xyz="0 0 0" rpy="0 0 0" />
-				<geometry>
-          				<!--<mesh filename="package://youbot_description/meshes/youbot_base/youbot_wheel.stl" />-->
-					<sphere radius="${wheel_radius}"/>
-        			</geometry>
-       				<material name="Orange" />
-      			</visual>
-      			<collision>
-        			<origin xyz="0 0 0" rpy="${M_PI/2} 0 0" />
-        			<geometry>
-        		       		<cylinder radius="${wheel_radius}" length="${wheel_radius}" />
-        	       		</geometry>
-      			</collision>
-    		</link>
-	<!-- extensions -->
-		<xacro:youbot_base_gazebo />
-		<xacro:youbot_base_transmission />
-	</xacro:macro>
+    <!-- sensors -->
+    <xacro:include filename="$(find youbot_description)/urdf/sensors/hokuyo_urg04_laser.urdf.xacro"/>
+    <xacro:include filename="$(find youbot_description)/urdf/youbot_base/base.gazebo.xacro" />
+    <xacro:include filename="$(find youbot_description)/urdf/youbot_base/base.transmission.xacro" />
+    <!-- simplified box collision geometry for base -->
+    <xacro:property name="base_size_x" value="0.570" />
+    <xacro:property name="base_size_y" value="0.360" />
+    <xacro:property name="base_size_z" value="0.100" />
+    <xacro:property name="base_mass" value="22.0" />
+    <xacro:property name="caster_offset_x" value="0.228"  />
+    <xacro:property name="caster_offset_y" value="0.158"  />
+    <xacro:property name="caster_offset_z" value="-0.034" />
+    <xacro:property name="caster_mass" value="0.1" />
+    <xacro:property name="wheel_offset_x" value="0.0"  />
+    <xacro:property name="wheel_offset_y" value="0.0"  />
+    <xacro:property name="wheel_offset_z" value="0.0" />
+    <xacro:property name="wheel_mass" value="0.4" />
+    <xacro:property name="wheel_radius" value="0.05" />
+    <xacro:property name="wheel_length" value="0.005" />
+    <xacro:property name="caster_joint_damping" value="1.0" />
+    <xacro:property name="caster_joint_friction" value="1.0" />
+    <xacro:property name="caster_joint_effort" value="30" />
+    <xacro:property name="caster_joint_velocity" value="10" />
+    <xacro:property name="caster_joint_safety_k_velocity" value="10.0" />
+    <xacro:property name="wheel_joint_damping" value="1.0" />
+    <xacro:property name="wheel_joint_friction" value="1.0" />
+    <xacro:property name="wheel_joint_effort" value="30" />
+    <xacro:property name="wheel_joint_velocity" value="10" />
+    <xacro:property name="wheel_joint_safety_k_velocity" value="10.0" />
+    <xacro:macro name="youbot_base" params="name">
+    <link name="${name}_footprint">
+        <inertial>
+            <mass value="0.1" />
+            <origin xyz="0 0 ${-base_size_z / 2.0}" rpy="0 0 0" />
+            <inertia ixx="1.0" ixy="0.0" ixz="0.0"
+            iyy="1.0" iyz="0.0" izz="1.0" />
+        </inertial>
+        <visual>
+            <origin xyz="0 0 0" rpy="0 0 0" />
+                <geometry>
+            <box size="0.001 0.001 0.001" />
+                </geometry>
+            <material name="Red" />
+        </visual>
+        <collision>
+            <origin xyz="0 0 ${-base_size_z / 2.0}" rpy="0 0 0" />
+            <geometry>
+                <box size="0.001 0.001 0.001" />
+            </geometry>
+        </collision>
+    </link>
+    <joint name="${name}_footprint_joint" type="fixed">
+        <origin xyz="0 0 0" rpy="0 0 0" />
+        <child link="${name}_link" />
+        <parent link="${name}_footprint"/>
+    </joint>
+    <link name="${name}_link">
+        <inertial>
+            <mass value="${base_mass}" />
+            <origin xyz="0 0 0" />
+            <inertia ixx="5.652232699207" ixy="-0.009719934438" ixz="1.293988226423"
+            iyy="5.669473158652" iyz="-0.007379583694" izz="3.683196351726" />
+        </inertial>
+        <visual>
+            <origin xyz="0 0 0" rpy="0 0 0" />
+            <geometry>
+            <mesh filename="package://youbot_description/meshes/youbot_base/base.dae"/>
+            </geometry>
+            <material name="DarkGrey"/>
+        </visual>
+        <collision>
+            <origin xyz="0 0 0" rpy="0 0 0" />
+            <geometry>
+            <!--<box size="${base_size_x} ${base_size_y} ${base_size_z}" />-->
+            <mesh filename="package://youbot_description/meshes/youbot_base/base_convex.dae"/>
+            </geometry>
+        </collision>
+    </link>
+    <!-- base laser front -->
+    <xacro:hokuyo_urg04_laser name="${name}_laser_front" parent="${name}" ros_topic="scan_front" update_rate="10" min_angle="-1.57" max_angle="1.57" >
+        <origin xyz="0.3 0 -0.03" rpy="0 0 0" />
+    </xacro:hokuyo_urg04_laser>
+    <!-- front left wheel -->
+    <joint name="caster_joint_fl" type="continuous">
+        <origin xyz="${caster_offset_x} ${caster_offset_y} ${caster_offset_z}" rpy="0 0 0" />
+        <axis xyz="0 0 1" />
+        <limit effort="${caster_joint_effort}" velocity="${caster_joint_velocity}"/>
+        <dynamics damping="${caster_joint_damping}" friction="${caster_joint_friction}" />
+        <safety_controller k_velocity="${caster_joint_safety_k_velocity}" />
+        <parent link="${name}_link"/>
+        <child link="caster_link_fl" />
+    </joint>
+    <link name="caster_link_fl">
+        <inertial>
+            <mass value="${caster_mass}" />
+            <origin xyz="0 0 0" />
+            <inertia  ixx="0.012411765597" ixy="-0.000711733678" ixz="0.00050272983"
+            iyy="0.015218160428" iyz="-0.000004273467" izz="0.011763977943" />
+        </inertial>
+    </link>
+    <joint name="wheel_joint_fl" type="continuous">
+        <axis xyz="0 1 0" />
+        <limit effort="${wheel_joint_effort}" velocity="${wheel_joint_velocity}"/>
+        <origin xyz="${wheel_offset_x} ${wheel_offset_y} ${wheel_offset_z}" rpy="0 0 0" />
+        <parent link="caster_link_fl"/>
+        <dynamics damping="${wheel_joint_damping}" friction="${wheel_joint_friction}" />
+        <safety_controller k_velocity="${wheel_joint_safety_k_velocity}" />
+        <child link="wheel_link_fl"/>
+    </joint>
+    <link name="wheel_link_fl">
+        <inertial>
+            <mass value="${wheel_mass}" />
+            <origin xyz="0 0 0" />
+            <inertia  ixx="0.012411765597" ixy="-0.000711733678" ixz="0.00050272983"
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
File: youbot_ws/src/ros_stacks/youbot-ros-pkg/youbot_common/youbot_description/urdf/youbot_gripper/limits.urdf.xacro (robot description, xacro)
@@ -1,9 +1,12 @@
 <?xml version="1.0"?>
-<robot>
+<robot  xmlns:sensor="http://playerstage.sourceforge.net/gazebo/xmlschema/#sensor"
+        xmlns:controller="http://playerstage.sourceforge.net/gazebo/xmlschema/#controller"
+        xmlns:interface="http://playerstage.sourceforge.net/gazebo/xmlschema/#interface"
+        xmlns:xacro="http://ros.org/wiki/xacro">
 	<!-- common properties -->
-	<property name="M_PI" value="3.1415926535897931" />
-        <property name="threshold" value="0.001" />
+	<xacro:property name="M_PI" value="3.1415926535897931" />
+    <xacro:property name="threshold" value="0.001" />
 	<!-- fingers limits, values are in meters -->
-	<property name="finger_joint" value="${0.023 / 2.0}" />
-	<property name="finger_joint_soft" value="${(0.023 - threshold) / 2.0}" />
+	<xacro:property name="finger_joint" value="${0.023 / 2.0}" />
+	<xacro:property name="finger_joint_soft" value="${(0.023 - threshold) / 2.0}" />
 </robot>
