Commit message: Introduce RealSense Plugin and added it to the simulation with aruco

File: youbot_ws/src/ros_stacks/youbot-ros-pkg/youbot_common/youbot_description/robots/youbot.urdf.xacro (robot description, xacro)
@@ -13,7 +13,9 @@
   <xacro:include filename="$(find youbot_description)/urdf/youbot_plate/plate.urdf.xacro" />
   <!-- youbot arm -->
-  <xacro:include filename="$(find youbot_description)/urdf/youbot_arm/arm.urdf.xacro"/>
+  <!-- <xacro:include filename="$(find youbot_description)/urdf/youbot_arm/arm.urdf.xacro"/> Xacro file for the arm-->
+  <xacro:include filename="$(find youbot_description)/urdf/youbot_arm/static_link.urdf.xacro"/>
   <!-- youbot gripper -->
-  <xacro:include filename="$(find youbot_description)/urdf/youbot_gripper/gripper.urdf.xacro" />
+  <!-- <xacro:include filename="$(find youbot_description)/urdf/youbot_gripper/gripper.urdf.xacro" /> -->
+   <xacro:include filename="$(find realsense2_description)/urdf/_d435.urdf.xacro"/>
   <!-- generic simulator_gazebo plugins for starting mechanism control, ros time, ros battery -->
   <xacro:include filename="$(find youbot_description)/gazebo/gazebo.urdf.xacro" />
@@ -33,9 +35,15 @@
     <origin xyz="-0.159 0 0.046" rpy="0 0 0" />
   </xacro:youbot_plate>
-  <xacro:youbot_arm name="arm" parent="base_link">
+  <xacro:youbot_static_link name="static_link" parent="base_link">
+    <origin xyz="0.143 0 0.046" rpy="0 0 0" />
+  </xacro:youbot_static_link>
+  <xacro:sensor_d435 name="camera" parent="static_link">
+    <origin xyz="0 0 0.25" rpy="0 0 0" />
+  </xacro:sensor_d435>
+  <!-- <xacro:youbot_arm name="arm" parent="base_link">
     <origin xyz="0.143 0 0.046" rpy="0 0 0" />
   </xacro:youbot_arm>
   <xacro:youbot_gripper name="gripper" parent="arm_link_5">
     <origin xyz="0 0 0" rpy="0 0 0" />
-  </xacro:youbot_gripper>
+  </xacro:youbot_gripper> -->
 </robot>

File: youbot_ws/src/ros_stacks/youbot-ros-pkg/youbot_common/youbot_description/urdf/materials.urdf.xacro (robot description, xacro)
@@ -1,7 +1,7 @@
 <?xml version="1.0"?>
 <robot>
-  <material name="Orange">
+  <!-- <material name="Orange">
     <color rgba="1.0 0.4 0.0 1.0"/>
-  </material>
+  </material> -->
   <material name="Grey">
     <color rgba="0.7 0.7 0.7 1.0"/>

File: youbot_ws/src/ros_stacks/youbot-ros-pkg/youbot_common/youbot_description/urdf/youbot_arm/arm.gazebo.xacro (robot description, xacro)
@@ -4,29 +4,33 @@
        xmlns:interface="http://playerstage.sourceforge.net/gazebo/xmlschema/#interface"
        xmlns:xacro="http://ros.org/wiki/xacro">
-	<xacro:macro name="youbot_arm_gazebo" params="name">
-		<gazebo reference="${name}_link_0">
+	<xacro:macro name="youbot_arm_gazebo">    <!--params="name"-->
+		<gazebo reference="youbot_static_link">
+			<!--<material value="youbot/Orange" /> -->
+			<turnGravityOff>false</turnGravityOff>
+		</gazebo>
+		<!--<gazebo reference="${name}_link_0">
 			<material value="youbot/DarkGrey" />
 			<turnGravityOff>false</turnGravityOff>
-		</gazebo>
-		<gazebo reference="${name}_link_1">
-			<!--<material value="youbot/Orange" />-->
+		</gazebo> -->
+		<!-- <gazebo reference="${name}_link_1">
+			 <material value="youbot/Orange" />
 			<turnGravityOff>false</turnGravityOff>
-		</gazebo>
-		<gazebo reference="${name}_link_2">
-			<!--<material value="youbot/Orange" />-->
+		</gazebo> -->
+		<!--<gazebo reference="${name}_link_2">
+			<material value="youbot/Orange" />
 			<turnGravityOff>false</turnGravityOff>
-		</gazebo>
-		<gazebo reference="${name}_link_3">
-			<!--<material value="youbot/Orange" />-->
+		</gazebo> -->
+		<!--<gazebo reference="${name}_link_3">
+			<material value="youbot/Orange" />
 			<turnGravityOff>false</turnGravityOff>
-		</gazebo>
-		<gazebo reference="${name}_link_4">
-			<!--<material value="youbot/Orange" />-->
+		</gazebo> -->
+		<!--<gazebo reference="${name}_link_4">
+			<material value="youbot/Orange" />
 			<turnGravityOff>false</turnGravityOff>
-		</gazebo>
-		<gazebo reference="${name}_link_5">
-			<!--<material value="youbot/DarkGrey" />-->
+		</gazebo> -->
+		<!--<gazebo reference="${name}_link_5">
+			<material value="youbot/DarkGrey" />
 			<turnGravityOff>false</turnGravityOff>
-		</gazebo>
+		</gazebo> -->
 	</xacro:macro>
 </robot>

Commit message: Added proportional controller for aruco-21 tracking with simulation parameters

File: youbot_ws/src/ros_stacks/youbot-ros-pkg/youbot_common/youbot_description/robots/youbot.urdf.xacro (robot description, xacro)
@@ -39,5 +39,5 @@
   </xacro:youbot_static_link>
   <xacro:sensor_d435 name="camera" parent="static_link">
-    <origin xyz="0 0 0.25" rpy="0 0 0" />
+    <origin xyz="0 0 0.125" rpy="0 0 0" />
   </xacro:sensor_d435>
   <!-- <xacro:youbot_arm name="arm" parent="base_link">

File: youbot_ws/src/ros_stacks/youbot-ros-pkg/youbot_common/youbot_description/urdf/youbot_arm/static_link.urdf.xacro (robot description, xacro)
@@ -4,5 +4,5 @@
     <xacro:include filename="$(find youbot_description)/urdf/youbot_arm/arm.gazebo.xacro" />
     <xacro:property name="static_link_radius" value="0.01" />
-    <xacro:property name="static_link_length" value="0.25" />
+    <xacro:property name="static_link_length" value="0.125" />
     <xacro:macro name = "youbot_static_link" params="parent name *origin">
         <!-- joint between base_link and arm_0_link -->
@@ -19,5 +19,5 @@
 			</inertial>
             <visual>
-				<origin xyz="0 0 0.125" rpy="0 0 0" />
+				<origin xyz="0 0 0.0625" rpy="0 0 0" />
 				<geometry>
 					<cylinder radius="${static_link_radius}" length="${static_link_length}"/>
